Commit message: add hotel stair world and b2 description

File: robots/go2w_description/xacro/gazebo.xacro (robot description, xacro)
@@ -25,5 +25,5 @@
     </gazebo> -->
     <!-- Show the trajectory of foot. You can add another trajectory about another foot. -->
-    <!-- <gazebo>
+    <gazebo>
         <plugin name="3dplot" filename="libLinkPlot3DPlugin.so">
             <frequency>100</frequency>
@@ -34,5 +34,5 @@
             </plot>
         </plugin>
-    </gazebo> -->
+    </gazebo>
     <gazebo>
         <plugin filename="libgazebo_ros_force.so" name="gazebo_ros_force">
@@ -98,5 +98,5 @@
     </gazebo>
     <!-- Visualization of Foot contacts. -->
-    <!-- <gazebo reference="FR_foot">
+    <gazebo reference="FR_foot">
         <visual>
             <plugin name="drawForcePlugin" filename="libunitreeDrawForcePlugin.so">
@@ -125,5 +125,5 @@
             </plugin>
         </visual>
-    </gazebo> -->
+    </gazebo>
     </xacro:if>
     <xacro:if value="${int(ros_version) == 2}">

File: robots/go2w_description/xacro/robot.xacro (robot description, xacro)
@@ -10,5 +10,5 @@
     <!-- Mount for VLP-16 LiDAR -->
     <joint name="vlp16_mount_joint" type="fixed">
-        <origin xyz="0.16143 0 0.12262" rpy="0 0.22689 0"/>
+        <origin xyz="0.14543 0 0.13928" rpy="0 0 0"/>
         <parent link="base_link"/>
         <child link="vlp16_link"/>
