Commit message: update livox imu

File: robots/go2_description/urdf/go2_description.urdf (robot description, URDF)
Before this commit: robot go2_description, 30 links, 29 joints
Links:
- added link livox_imu_link, mass 0
Joints:
- added joint livox_imu_joint: type fixed, parent base, child livox_imu_link, origin xyz=0.16143 0 0.12262 rpy=0 0.22689 0, axis 0 0 0

File: robots/go2_description/xacro/gazebo.xacro (robot description, xacro)
@@ -133,4 +133,72 @@
             <namespace>/</namespace>
             <remapping>~/out:=imu</remapping>
+          </ros>
+          <initial_orientation_as_reference>false</initial_orientation_as_reference>
+        </plugin>
+        <always_on>true</always_on>
+        <update_rate>100</update_rate>
+        <visualize>true</visualize>
+        <imu>
+          <angular_velocity>
+            <x>
+              <noise type="gaussian">
+                <mean>0.0</mean>
+                <stddev>2e-4</stddev>
+                <bias_mean>0.0000075</bias_mean>
+                <bias_stddev>0.0000008</bias_stddev>
+              </noise>
+            </x>
+            <y>
+              <noise type="gaussian">
+                <mean>0.0</mean>
+                <stddev>2e-4</stddev>
+                <bias_mean>0.0000075</bias_mean>
+                <bias_stddev>0.0000008</bias_stddev>
+              </noise>
+            </y>
+            <z>
+              <noise type="gaussian">
+                <mean>0.0</mean>
+                <stddev>2e-4</stddev>
+                <bias_mean>0.0000075</bias_mean>
+                <bias_stddev>0.0000008</bias_stddev>
+              </noise>
+            </z>
+          </angular_velocity>
+          <linear_acceleration>
+            <x>
+              <noise type="gaussian">
+                <mean>0.0</mean>
+                <stddev>1.7e-2</stddev>
+                <bias_mean>0.1</bias_mean>
+                <bias_stddev>0.001</bias_stddev>
+              </noise>
+            </x>
+            <y>
+              <noise type="gaussian">
+                <mean>0.0</mean>
+                <stddev>1.7e-2</stddev>
+                <bias_mean>0.1</bias_mean>
+                <bias_stddev>0.001</bias_stddev>
+              </noise>
+            </y>
+            <z>
+              <noise type="gaussian">
+                <mean>0.0</mean>
+                <stddev>1.7e-2</stddev>
+                <bias_mean>0.1</bias_mean>
+                <bias_stddev>0.001</bias_stddev>
+              </noise>
+            </z>
+          </linear_acceleration>
+        </imu>
+      </sensor>
+    </gazebo>
+    <gazebo reference="livox_imu_link">
+      <sensor name="livox_imu_sensor" type="imu">
+      <plugin filename="libgazebo_ros_imu_sensor.so" name="livox_imu_plugin">
+          <ros>
+            <namespace>/</namespace>
+            <remapping>~/out:=livox/imu</remapping>
           </ros>
           <initial_orientation_as_reference>false</initial_orientation_as_reference>

File: robots/go2_description/xacro/robot.xacro (robot description, xacro)
@@ -4,6 +4,6 @@
     <xacro:include filename="$(find go2_description)/xacro/gazebo.xacro"/>
     <xacro:include filename="$(find ros2_livox_simulation)/urdf/mid360.xacro"/>
-    <xacro:mid360 name="livox_frame" parent="imu_link" topic="livox/lidar">
-        <origin xyz="0.1870 0 0.0803" rpy="0 0.22689 0"/>
+    <xacro:mid360 name="livox_frame" parent="base" topic="livox/lidar">
+        <origin xyz="0.16143 0 0.12262" rpy="0 0.22689 0"/>
     </xacro:mid360>
 </robot>

File: robots/go2w_description/urdf/go2w_description.urdf (robot description, URDF)
Before this commit: robot go2w_description, 34 links, 33 joints
Links:
- added link livox_imu_link, mass 0
Joints:
- added joint livox_imu_joint: type fixed, parent base, child livox_imu_link, origin xyz=0.16143 0 0.12262 rpy=0 0.22689 0, axis 0 0 0

File: robots/go2w_description/xacro/gazebo.xacro (robot description, xacro)
@@ -134,4 +134,72 @@
             <namespace>/</namespace>
             <remapping>~/out:=imu</remapping>
+          </ros>
+          <initial_orientation_as_reference>false</initial_orientation_as_reference>
+        </plugin>
+        <always_on>true</always_on>
+        <update_rate>100</update_rate>
+        <visualize>true</visualize>
+        <imu>
+          <angular_velocity>
+            <x>
+              <noise type="gaussian">
+                <mean>0.0</mean>
+                <stddev>2e-4</stddev>
+                <bias_mean>0.0000075</bias_mean>
+                <bias_stddev>0.0000008</bias_stddev>
+              </noise>
+            </x>
+            <y>
+              <noise type="gaussian">
+                <mean>0.0</mean>
+                <stddev>2e-4</stddev>
+                <bias_mean>0.0000075</bias_mean>
+                <bias_stddev>0.0000008</bias_stddev>
+              </noise>
+            </y>
+            <z>
+              <noise type="gaussian">
+                <mean>0.0</mean>
+                <stddev>2e-4</stddev>
+                <bias_mean>0.0000075</bias_mean>
+                <bias_stddev>0.0000008</bias_stddev>
+              </noise>
+            </z>
+          </angular_velocity>
+          <linear_acceleration>
+            <x>
+              <noise type="gaussian">
+                <mean>0.0</mean>
+                <stddev>1.7e-2</stddev>
+                <bias_mean>0.1</bias_mean>
+                <bias_stddev>0.001</bias_stddev>
+              </noise>
+            </x>
+            <y>
+              <noise type="gaussian">
+                <mean>0.0</mean>
+                <stddev>1.7e-2</stddev>
+                <bias_mean>0.1</bias_mean>
+                <bias_stddev>0.001</bias_stddev>
+              </noise>
+            </y>
+            <z>
+              <noise type="gaussian">
+                <mean>0.0</mean>
+                <stddev>1.7e-2</stddev>
+                <bias_mean>0.1</bias_mean>
+                <bias_stddev>0.001</bias_stddev>
+              </noise>
+            </z>
+          </linear_acceleration>
+        </imu>
+      </sensor>
+    </gazebo>
+    <gazebo reference="livox_imu_link">
+      <sensor name="livox_imu_sensor" type="imu">
+      <plugin filename="libgazebo_ros_imu_sensor.so" name="livox_imu_plugin">
+          <ros>
+            <namespace>/</namespace>
+            <remapping>~/out:=livox/imu</remapping>
           </ros>
           <initial_orientation_as_reference>false</initial_orientation_as_reference>

File: robots/go2w_description/xacro/robot.xacro (robot description, xacro)
@@ -4,6 +4,6 @@
     <xacro:include filename="$(find go2w_description)/xacro/gazebo.xacro"/>
     <xacro:include filename="$(find ros2_livox_simulation)/urdf/mid360.xacro"/>
-    <xacro:mid360 name="livox_frame" parent="imu_link" topic="livox/lidar">
-        <origin xyz="0.1870 0 0.0803" rpy="0 0.22689 0"/>
+    <xacro:mid360 name="livox_frame" parent="base" topic="livox/lidar">
+        <origin xyz="0.16143 0 0.12262" rpy="0 0.22689 0"/>
     </xacro:mid360>
 </robot>

Commit message: Replace mid360 with Velodyne in go2 description, remove Livox, and add hotel world

File: robots/go2_description/urdf/go2_description.urdf (robot description, URDF)
Before this commit: robot go2_description, 31 links, 30 joints
Links:
- removed link base
- added link base_link; visual box size=0.001 0.001 0.001
Joints:
- joint floating_base: parent base -> base_link
- joint livox_imu_joint: parent base -> base_link

File: robots/go2_description/xacro/gazebo.xacro (robot description, xacro)
@@ -294,5 +294,5 @@
     </gazebo>
     </xacro:if>
-    <gazebo reference="base">
+    <gazebo reference="base_link">
         <turnGravityOff>false</turnGravityOff>
     </gazebo>

File: robots/go2_description/xacro/robot.xacro (robot description, xacro)
@@ -3,7 +3,26 @@
     <xacro:include filename="$(find go2_description)/urdf/go2_description.urdf"/>
     <xacro:include filename="$(find go2_description)/xacro/gazebo.xacro"/>
-    <xacro:include filename="$(find ros2_livox_simulation)/urdf/mid360.xacro"/>
-    <xacro:mid360 name="livox_frame" parent="base" topic="livox/lidar">
+    <!-- LASER SCAN-->
+    <xacro:include filename="$(find velodyne_description)/urdf/VLP-16.urdf.xacro" />
+    <xacro:VLP-16 parent="vlp16_link" name="vlp16" tf_prefix="" topic="/velodyne_points" organize_cloud="false" hz="10" lasers="16" samples="1000" collision_range="0.3" min_range="0.9" max_range="30.0" noise="0.008" min_angle="-${M_PI}" max_angle="${M_PI}" gpu="true">
+        <origin xyz="0.0 0.0 0.0" rpy="0 0 0"/>
+    </xacro:VLP-16>
+    <!-- Mount for VLP-16 LiDAR -->
+    <joint name="vlp16_mount_joint" type="fixed">
+        <origin xyz="0.16143 0 0.12262" rpy="0 0 0"/>
+        <parent link="base_link"/>
+        <child link="vlp16_link"/>
+    </joint>
+    <link name="vlp16_link">
+        <visual>
+            <origin xyz="0.0 0.0 0.0" rpy="0 0 0"/>
+            <geometry>
+                <mesh filename="file://$(find velodyne_description)/meshes/VLP16_scan.dae" />
+            </geometry>
+        </visual>
+    </link>
+    <!-- <xacro:include filename="$(find ros2_livox_simulation)/urdf/mid360.xacro"/>
+    <xacro:mid360 name="livox_frame" parent="base_link" topic="livox/lidar">
         <origin xyz="0.16143 0 0.12262" rpy="0 0.22689 0"/>
-    </xacro:mid360>
+    </xacro:mid360> -->
 </robot>

File: robots/go2w_description/urdf/go2w_description.urdf (robot description, URDF)
Before this commit: robot go2w_description, 35 links, 34 joints
Links:
- removed link base
- added link base_link; visual box size=0.001 0.001 0.001
Joints:
- joint floating_base: parent base -> base_link
- joint livox_imu_joint: parent base -> base_link

File: robots/go2w_description/xacro/gazebo.xacro (robot description, xacro)
@@ -296,5 +296,5 @@
     </gazebo>
     </xacro:if>
-    <gazebo reference="base">
+    <gazebo reference="base_link">
         <material>Gazebo/Green</material>
         <turnGravityOff>false</turnGravityOff>

File: robots/go2w_description/xacro/robot.xacro (robot description, xacro)
@@ -3,7 +3,22 @@
     <xacro:include filename="$(find go2w_description)/urdf/go2w_description.urdf"/>
     <xacro:include filename="$(find go2w_description)/xacro/gazebo.xacro"/>
-    <xacro:include filename="$(find ros2_livox_simulation)/urdf/mid360.xacro"/>
-    <xacro:mid360 name="livox_frame" parent="base" topic="livox/lidar">
+    <!-- LASER SCAN-->
+    <xacro:include filename="$(find velodyne_description)/urdf/VLP-16.urdf.xacro" />
+    <xacro:VLP-16 parent="vlp16_link" name="vlp16" tf_prefix="" topic="/velodyne_points" organize_cloud="false" hz="10" lasers="16" samples="1000" collision_range="0.3" min_range="0.9" max_range="30.0" noise="0.008" min_angle="-${M_PI}" max_angle="${M_PI}" gpu="true">
+        <origin xyz="0.0 0.0 0.0" rpy="0 0 0"/>
+    </xacro:VLP-16>
+    <!-- Mount for VLP-16 LiDAR -->
+    <joint name="vlp16_mount_joint" type="fixed">
         <origin xyz="0.16143 0 0.12262" rpy="0 0.22689 0"/>
-    </xacro:mid360>
+        <parent link="base_link"/>
+        <child link="vlp16_link"/>
+    </joint>
+    <link name="vlp16_link">
+        <visual>
+            <origin xyz="0.0 0.0 0.0" rpy="0 0 0"/>
+            <geometry>
+                <mesh filename="file://$(find velodyne_description)/meshes/VLP16_scan.dae" />
+            </geometry>
+        </visual>
+    </link>
 </robot>

Commit message: add elevator plugin

File: robots/go2_description/urdf/go2_description.urdf (robot description, URDF)
Before this commit: robot go2_description, 31 links, 30 joints
Joints:
- joint livox_imu_joint: origin xyz=0.16143 0 0.12262 rpy=0 0.22689 0 -> xyz=-0.02557 0 0.04232 rpy=0 0 0

File: robots/go2_description/xacro/robot.xacro (robot description, xacro)
@@ -10,5 +10,5 @@
     <!-- Mount for VLP-16 LiDAR -->
     <joint name="vlp16_mount_joint" type="fixed">
-        <origin xyz="0.16143 0 0.12262" rpy="0 0 0"/>
+        <origin xyz="0.14543 0 0.13928" rpy="0 0 0"/>
         <parent link="base_link"/>
         <child link="vlp16_link"/>
