Commit message: revise b2_description(lidar), worlds

File: robots/b2_description/urdf/b2_description.urdf (robot description, URDF)
Before this commit: robot b2_description, 26 links, 25 joints
Links:
- link trunk: geometry collision box size=0.5 0.28 0.15; visual mesh filename=package://b2_description/meshes/trunk2.dae
- link vlp16_link: geometry collision cylinder length=0.16 radius=0.076; visual mesh filename=file://$(find velodyne_description)/meshes/VLP16_scan.dae
Joints:
- removed joint vlp16_joint
- added joint vlp16_mount_joint: type fixed, parent base_link, child vlp16_link, origin xyz=0.34918 0 0.17851 rpy=0 0 0, axis 0 0 0

File: robots/b2_description/xacro/robot.xacro (robot description, xacro)
@@ -3,4 +3,8 @@
     <xacro:include filename="$(find b2_description)/xacro/gazebo.xacro"/>
     <xacro:include filename="$(find b2_description)/urdf/b2_description.urdf"/>
+    <xacro:include filename="$(find velodyne_description)/urdf/VLP-16.urdf.xacro" />
+    <xacro:VLP-16 parent="vlp16_link" name="vlp16" tf_prefix="" topic="/velodyne_points" organize_cloud="false" hz="10" lasers="16" samples="1000" collision_range="0.3" min_range="0.9" max_range="30.0" noise="0.008" min_angle="-${M_PI}" max_angle="${M_PI}" gpu="true">
+        <origin xyz="0.0 0.0 0.0" rpy="0 0 0"/>
+    </xacro:VLP-16>
     <!-- Rotor related joint and link is only for demonstrate location. -->
     <!-- Actually, the rotor will rotate and the joint is not fixed. Reduction ratio should be considered. -->
